File: CAN_Controller_Transceiver.kicad_sch (KiCad schematic)
At the start: 31 parts, among them J11 Screw_Terminal_01x02, J12 DB9_Male, SW1 SW_SPDT, U1 MCP2515-xSO, U2 MCP2551-I-SN, U3 LD1117S50TR_SOT223, Y1 8MHz Crystal

Commit message: Complete Board (1)
Connections:
- net IO10: now also U1.4 (~{TX0RTS}); no longer U1.5 (~{TX1RTS})
- net IO11: now also U1.3 (CLKOUT/SOF); no longer U1.6 (~{TX2RTS})
- net IO17: now also U2.8 (Rs); no longer U1.10 (~{RX1BF})
- net IO18: now also U1.10 (~{RX1BF}); no longer U1.11 (~{RX0BF})
- net IO19: now also U1.11 (~{RX0BF}); no longer R6.1, U1.12 (~{INT})
- net IO20: now also R6.1, U1.12 (~{INT}); no longer U2.8 (Rs)
- net IO8: now also U1.6 (~{TX2RTS}); no longer U1.3 (CLKOUT/SOF)
- net IO9: now also U1.5 (~{TX1RTS}); no longer U1.4 (~{TX0RTS})
Changed lines of the file:
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@@
     (effects (font (size 1.27 1.27)) (justify left bottom))
   )
-  (label "IO10" (at 97.79 72.39 0)
-    (effects (font (size 1.27 1.27)) (justify left bottom))
-  )
-  (label "IO11" (at 97.79 74.93 0)
+  (label "IO9" (at 97.79 72.39 0)
+    (effects (font (size 1.27 1.27)) (justify left bottom))
+  )
+  (label "IO8" (at 97.79 74.93 0)
     (effects (font (size 1.27 1.27)) (justify left bottom))
   )
@@
     (effects (font (size 1.27 1.27)) (justify left bottom))
   )
-  (label "IO8" (at 97.79 59.69 0)
-    (effects (font (size 1.27 1.27)) (justify left bottom))
-  )
-  (label "IO9" (at 97.79 69.85 0)
-    (effects (font (size 1.27 1.27)) (justify left bottom))
-  )
-  (label "IO20" (at 152.4 58.42 0)
+  (label "IO11" (at 97.79 59.69 0)
+    (effects (font (size 1.27 1.27)) (justify left bottom))
+  )
+  (label "IO10" (at 97.79 69.85 0)
+    (effects (font (size 1.27 1.27)) (justify left bottom))
+  )
+  (label "IO17" (at 152.4 58.42 0)
     (effects (font (size 1.27 1.27)) (justify left bottom))
   )
@@
     (effects (font (size 1.27 1.27)) (justify left bottom))
   )
-  (label "IO19" (at 97.79 62.23 0)
+  (label "IO20" (at 97.79 62.23 0)
     (effects (font (size 1.27 1.27)) (justify left bottom))
   )
@@
     (effects (font (size 1.27 1.27)) (justify left bottom))
   )
-  (label "IO17" (at 97.79 67.31 0)
+  (label "IO18" (at 97.79 67.31 0)
     (effects (font (size 1.27 1.27)) (justify left bottom))
   )
@@
     (effects (font (size 1.27 1.27)) (justify left bottom))
   )
-  (label "IO18" (at 97.79 64.77 0)
-    (effects (font (size 1.27 1.27)) (justify left bottom))
-  )
-  (global_label "IO19" (shape input) (at 220.98 69.85 180) (fields_autoplaced)
+  (label "IO19" (at 97.79 64.77 0)
+    (effects (font (size 1.27 1.27)) (justify left bottom))
+  )
+  (global_label "IO20" (shape input) (at 220.98 69.85 180) (fields_autoplaced)
     (effects (font (size 1.27 1.27)) (justify right))
     (property "Intersheet References" "${INTERSHEET_REFS}" (id 0) (at 214.2126 69.7706 0)
@@
       (effects (font (size 1.27 1.27)) hide)
     )
-    (property "Datasheet" "~" (id 3) (at 44.45 168.91 0)
+    (property "Datasheet" "https://www.digikey.com/en/products/detail/cui-devices/TB006-508-02BE/10064115" (id 3) (at 44.45 168.91 0)
       (effects (font (size 1.27 1.27)) hide)
     )
@@
       (effects (font (size 1.27 1.27)) hide)
     )
-    (property "Datasheet" "~" (id 3) (at 172.72 104.14 0)
-      (effects (font (size 1.27 1.27)) hide)
-    )
+    (property "Datasheet" "https://www.digikey.com/en/products/detail/eao/09-03290-01/8733106" (id 3) (at 172.72 104.14 0)
+      (effects (font (size 1.27 1.27)) hide)
+    )
